File: Kicad/PCMCIA_SRAM.sch (KiCad schematic (older format))
At the start: 21 parts, among them J1 PCMCIA, J2 JTAG, U1 SPX3819M5-L-3-3, U2 XC9536XL-VQ44, U3 CY62177ESL-55ZXI, U4 CY62167ELL-45ZXI

Commit message: v1.0 KiCAD files, D15/A0 bypass by default
Parts:
- JP1, JP3: footprint Jumper:SolderJumper-2_P1.3mm_Bridged_RoundedPad1.0x1.5mm -> Jumper:SolderJumper-2_P1.3mm_Open_RoundedPad1.0x1.5mm; symbol Jumper:SolderJumper_2_Bridged -> Jumper:SolderJumper_2_Open
- JP2: footprint Jumper:SolderJumper-2_P1.3mm_Open_RoundedPad1.0x1.5mm -> Jumper:SolderJumper-2_P1.3mm_Bridged_RoundedPad1.0x1.5mm; symbol Jumper:SolderJumper_2_Open -> Jumper:SolderJumper_2_Bridged
Connections:
- net +5V: now also JP7.1 (A); no longer JP7.3 (B)
- net _BYTE_A: now also JP7.3 (B); no longer JP7.1 (A)
Other:
- note added: "Odd-byte-low feature:\nThe PCMCIA 8bit feature, which makes the "Odd byte" available on D7:D0, is not necessary for Amiga computers.\n- To bypass the 8bit feature, close "D15 direct", open the two other links, and tie _BYTE to 5V. This is the default.\n\nFor other systems:\nNot sure if dynamically changing the BYTE# signal will work, and if the IO15_Axx signal will effectively select\nthe correct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"
- note removed: "WARNING : the whole thing is untested and moght not work at all !\nNot sure if the PCMCIA 8bit feature, which makes the "Odd byte" available on D7:D0, is necessary in our case.\nNot sure if dynamically changing the BYTE# signal will work, and if the IO15_Axx signal will effectively select\nthe correct bytes. According to Cypress this should not work : https://community.cypress.com/message/231471\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"
Changed lines of the file:
@@
 Title "PCMCIA SRAM"
 Date "2020-04-19"
-Rev "v0.1"
+Rev "v1.0"
 Comp "FLACO 2019 - Creative Commons Attribution-ShareAlike 4.0 license"
 Comment1 "Inspired by Sakura designs https://github.com/Sakura-IT/ppa-pcmcia-sram"
@@
 4MB
 $Comp
-L Jumper:SolderJumper_2_Open JP2
+L Jumper:SolderJumper_2_Bridged JP2
 U 1 1 5EA351D7
 P 5450 7000
 F 0 "JP2" H 5450 7205 50  0000 C CNN
 F 1 "D15 direct" H 5450 7114 50  0000 C CNN
-F 2 "Jumper:SolderJumper-2_P1.3mm_Open_RoundedPad1.0x1.5mm" H 5450 7000 50  0001 C CNN
+F 2 "Jumper:SolderJumper-2_P1.3mm_Bridged_RoundedPad1.0x1.5mm" H 5450 7000 50  0001 C CNN
 F 3 "~" H 5450 7000 50  0001 C CNN
 	1    5450 7000
@@
 $EndComp
 $Comp
-L Jumper:SolderJumper_2_Bridged JP3
+L Jumper:SolderJumper_2_Open JP3
 U 1 1 5EA362F2
 P 5800 7250
 F 0 "JP3" V 5754 7318 50  0000 L CNN
 F 1 "D15 A0" V 5845 7318 50  0000 L CNN
-F 2 "Jumper:SolderJumper-2_P1.3mm_Bridged_RoundedPad1.0x1.5mm" H 5800 7250 50  0001 C CNN
+F 2 "Jumper:SolderJumper-2_P1.3mm_Open_RoundedPad1.0x1.5mm" H 5800 7250 50  0001 C CNN
 F 3 "~" H 5800 7250 50  0001 C CNN
 	1    5800 7250
@@
 $EndComp
 $Comp
-L Jumper:SolderJumper_2_Bridged JP1
+L Jumper:SolderJumper_2_Open JP1
 U 1 1 5EA3899D
 P 5100 7250
 F 0 "JP1" V 5054 7318 50  0000 L CNN
 F 1 "D15 pcmcia" V 5145 7318 50  0000 L CNN
-F 2 "Jumper:SolderJumper-2_P1.3mm_Bridged_RoundedPad1.0x1.5mm" H 5100 7250 50  0001 C CNN
+F 2 "Jumper:SolderJumper-2_P1.3mm_Open_RoundedPad1.0x1.5mm" H 5100 7250 50  0001 C CNN
 F 3 "~" H 5100 7250 50  0001 C CNN
 	1    5100 7250
@@
 	1    0    0    -1
 $EndComp
-$Comp
-L Jumper:SolderJumper_3_Bridged12 JP7
-U 1 1 5E9C4B12
-P 6650 7300
-F 0 "JP7" V 6696 7368 50  0000 L CNN
-F 1 "_BYTE" V 6605 7368 50  0000 L CNN
-F 2 "Jumper:SolderJumper-3_P1.3mm_Bridged12_RoundedPad1.0x1.5mm" H 6650 7300 50  0001 C CNN
-F 3 "~" H 6650 7300 50  0001 C CNN
-	1    6650 7300
-	0    1    -1   0
-$EndComp
 Text Label 6650 7500 2    50   ~ 0
 _BYTE_A
@@
 NoConn ~ 5150 4000
 Wire Notes Line
-	6950 6550 6950 7750
+	6950 6450 6950 7750
 Wire Notes Line
 	6950 7750 500  7750
 Wire Notes Line
-	500  7750 500  6550
+	500  7750 500  6450
 Wire Notes Line
-	500  6550 6950 6550
+	500  6450 6950 6450
 Text Notes 4250 1800 0    50   ~ 0
 CPLD logic
@@
 CPLD programming
 Text Notes 550  7650 0    50   ~ 0
-WARNING : the whole thing is untested and moght not work at all !\nNot sure if the PCMCIA 8bit feature, which makes the "Odd byte" available on D7:D0, is necessary in our case.\nNot sure if dynamically changing the BYTE# signal will work, and if the IO15_Axx signal will effectively select\nthe correct bytes. According to Cypress this should not work : https://community.cypress.com/message/231471\n- To bypass the 8bit feature, close "D15 direct" and open the two other links, and tie _BYTE to 5V\n- To try the workaround, open "D15 direct" and close the other links, and connect _BYTE to the CPLD\nWhen processed by the CPLD :\n- In 8 bit mode (_CE1=0 & _CE2=1 & A0=1), _BYTE=0, D15_A0=1, and D15=Z\n- In 16 bit mode,\n    - _BYTE=1,\n    - D15 is output to D15_A0 when _WE=0,\n    - D15_A0 is output to D15 when _OE=0 & CE_SINGLE=1 & _CE2=0
+Odd-byte-low feature:\nThe PCMCIA 8bit feature, which makes the "Odd byte" available on D7:D0, is not necessary for Amiga computers.\n- To bypass the 8bit feature, close "D15 direct", open the two other links, and tie _BYTE to 5V. This is the default.\n\nFor other systems:\nNot sure if dynamically changing the BYTE# signal will work, and if the IO15_Axx signal will effectively select\nthe correct bytes. According to Cypress this should not work : https://community.cypress.com/message/231471\n- To try the workaround, open "D15 direct" and close the other links, and connect _BYTE to the CPLD\nWhen processed by the CPLD :\n- In 8 bit mode (_CE1=0 & _CE2=1 & A0=1), _BYTE=0, D15_A0=1, and D15=Z\n- In 16 bit mode,\n    - _BYTE=1,\n    - D15 is output to D15_A0 when _WE=0,\n    - D15_A0 is output to D15 when _OE=0 & CE_SINGLE=1 & _CE2=0
 $Comp
 L Mechanical:Fiducial FID1
@@
 	1    0    0    -1
 $EndComp
+$Comp
+L Jumper:SolderJumper_3_Bridged12 JP7
+U 1 1 5E9C4B12
+P 6650 7300
+F 0 "JP7" V 6696 7368 50  0000 L CNN
+F 1 "_BYTE" V 6605 7368 50  0000 L CNN
+F 2 "Jumper:SolderJumper-3_P1.3mm_Bridged12_RoundedPad1.0x1.5mm" H 6650 7300 50  0001 C CNN
+F 3 "~" H 6650 7300 50  0001 C CNN
+	1    6650 7300
+	0    1    1    0
+$EndComp
 $EndSCHEMATC

Commit message: Made pads shorter on PCMCIA connector. Corrected license to CC-BY-NC-SA.
Parts:
- added FID2: Logo, Sassa:PIC_Cassepanards_GS, symbol Mechanical:Fiducial
- added U11: XC6206PxxxMR, Package_TO_SOT_SMD:SOT-23, symbol Regulator_Linear:XC6206PxxxMR
- FID1: footprint Sassa:CC_BY_SA_long_silkscreen_14x5.5mm -> Sassa:CC_BY_NC_SA_square_silkscreen
- J1: footprint Sassa:pcmcia -> Sassa:PCMCIA_female_edge_connector
Connections:
- net +3V3: now also U11.2 (VO)
- net +5V: now also U11.3 (VI)
- net GND: now also U11.1 (GND)
Other:
- note added: "alternative footprint"
- moved on the sheet: C3, C4, C5, C6, C7
Changed lines of the file:
@@
 F 0 "J1" H 2300 5517 50  0000 C CNN
 F 1 "PCMCIA" H 2300 5426 50  0000 C CNN
-F 2 "Sassa:pcmcia" H 2250 3700 50  0001 C CNN
+F 2 "Sassa:PCMCIA_female_edge_connector" H 2250 3700 50  0001 C CNN
 F 3 "~" H 2250 3700 50  0001 C CNN
 	1    2250 3700
@@
 L Device:C_Small C3
 U 1 1 5E9B3B63
-P 4050 1200
-F 0 "C3" H 4142 1246 50  0000 L CNN
-F 1 "100n" H 4142 1155 50  0000 L CNN
-F 2 "Capacitor_SMD:C_0805_2012Metric" H 4050 1200 50  0001 C CNN
-F 3 "~" H 4050 1200 50  0001 C CNN
-	1    4050 1200
+P 5300 1200
+F 0 "C3" H 5392 1246 50  0000 L CNN
+F 1 "100n" H 5392 1155 50  0000 L CNN
+F 2 "Capacitor_SMD:C_0805_2012Metric" H 5300 1200 50  0001 C CNN
+F 3 "~" H 5300 1200 50  0001 C CNN
+	1    5300 1200
 	1    0    0    -1
 $EndComp
@@
 L Device:C_Small C5
 U 1 1 5E9B4077
-P 4850 1200
-F 0 "C5" H 4942 1246 50  0000 L CNN
-F 1 "100n" H 4942 1155 50  0000 L CNN
-F 2 "Capacitor_SMD:C_0805_2012Metric" H 4850 1200 50  0001 C CNN
-F 3 "~" H 4850 1200 50  0001 C CNN
-	1    4850 1200
+P 6100 1200
+F 0 "C5" H 6192 1246 50  0000 L CNN
+F 1 "100n" H 6192 1155 50  0000 L CNN
+F 2 "Capacitor_SMD:C_0805_2012Metric" H 6100 1200 50  0001 C CNN
+F 3 "~" H 6100 1200 50  0001 C CNN
+	1    6100 1200
 	1    0    0    -1
 $EndComp
@@
 L power:+5V #PWR012
 U 1 1 5E9B4616
-P 4050 1100
-F 0 "#PWR012" H 4050 950 50  0001 C CNN
-F 1 "+5V" H 4065 1273 50  0000 C CNN
-F 2 "" H 4050 1100 50  0001 C CNN
-F 3 "" H 4050 1100 50  0001 C CNN
-	1    4050 1100
+P 5300 1100
+F 0 "#PWR012" H 5300 950 50  0001 C CNN
+F 1 "+5V" H 5315 1273 50  0000 C CNN
+F 2 "" H 5300 1100 50  0001 C CNN
+F 3 "" H 5300 1100 50  0001 C CNN
+	1    5300 1100
 	1    0    0    -1
 $EndComp
@@
 L Device:C_Small C4
 U 1 1 5E9B8FEF
-P 4400 1200
-F 0 "C4" H 4492 1246 50  0000 L CNN
-F 1 "100n" H 4492 1155 50  0000 L CNN
-F 2 "Capacitor_SMD:C_0805_2012Metric" H 4400 1200 50  0001 C CNN
-F 3 "~" H 4400 1200 50  0001 C CNN
-	1    4400 1200
+P 5650 1200
+F 0 "C4" H 5742 1246 50  0000 L CNN
+F 1 "100n" H 5742 1155 50  0000 L CNN
+F 2 "Capacitor_SMD:C_0805_2012Metric" H 5650 1200 50  0001 C CNN
+F 3 "~" H 5650 1200 50  0001 C CNN
+	1    5650 1200
 	1    0    0    -1
 $EndComp
@@
 L power:GND #PWR013
 U 1 1 5E9B9AEF
-P 4050 1300
-F 0 "#PWR013" H 4050 1050 50  0001 C CNN
-F 1 "GND" H 4055 1127 50  0000 C CNN
-F 2 "" H 4050 1300 50  0001 C CNN
-F 3 "" H 4050 1300 50  0001 C CNN
-	1    4050 1300
-	1    0    0    -1
-$EndComp
-Wire Wire Line
-	4400 1100 4050 1100
-Connection ~ 4050 1100
-Wire Wire Line
-	4400 1300 4050 1300
-Connection ~ 4050 1300
+P 5300 1300
+F 0 "#PWR013" H 5300 1050 50  0001 C CNN
+F 1 "GND" H 5305 1127 50  0000 C CNN
+F 2 "" H 5300 1300 50  0001 C CNN
+F 3 "" H 5300 1300 50  0001 C CNN
+	1    5300 1300
+	1    0    0    -1
+$EndComp
+Wire Wire Line
+	5650 1100 5300 1100
+Connection ~ 5300 1100
+Wire Wire Line
+	5650 1300 5300 1300
+Connection ~ 5300 1300
 $Comp
 L power:+3.3V #PWR016
 U 1 1 5E9BB2E8
-P 4850 1100
-F 0 "#PWR016" H 4850 950 50  0001 C CNN
-F 1 "+3.3V" H 4865 1273 50  0000 C CNN
-F 2 "" H 4850 1100 50  0001 C CNN
-F 3 "" H 4850 1100 50  0001 C CNN
-	1    4850 1100
+P 6100 1100
+F 0 "#PWR016" H 6100 950 50  0001 C CNN
+F 1 "+3.3V" H 6115 1273 50  0000 C CNN
+F 2 "" H 6100 1100 50  0001 C CNN
+F 3 "" H 6100 1100 50  0001 C CNN
+	1    6100 1100
 	1    0    0    -1
 $EndComp
@@
 L power:GND #PWR017
 U 1 1 5E9BB97B
-P 4850 1300
-F 0 "#PWR017" H 4850 1050 50  0001 C CNN
-F 1 "GND" H 4855 1127 50  0000 C CNN
-F 2 "" H 4850 1300 50  0001 C CNN
-F 3 "" H 4850 1300 50  0001 C CNN
-	1    4850 1300
+P 6100 1300
+F 0 "#PWR017" H 6100 1050 50  0001 C CNN
+F 1 "GND" H 6105 1127 50  0000 C CNN
+F 2 "" H 6100 1300 50  0001 C CNN
+F 3 "" H 6100 1300 50  0001 C CNN
+	1    6100 1300
 	1    0    0    -1
 $EndComp
@@
 L Device:C_Small C6
 U 1 1 5E9BBD76
-P 5200 1200
-F 0 "C6" H 5292 1246 50  0000 L CNN
-F 1 "100n" H 5292 1155 50  0000 L CNN
-F 2 "Capacitor_SMD:C_0805_2012Metric" H 5200 1200 50  0001 C CNN
-F 3 "~" H 5200 1200 50  0001 C CNN
-	1    5200 1200
-	1    0    0    -1
-$EndComp
-Wire Wire Line
-	5200 1100 4850 1100
-Connection ~ 4850 1100
-Wire Wire Line
-	5200 1300 4850 1300
-Connection ~ 4850 1300
-Text Notes 4000 850  0    50   ~ 0
+P 6450 1200
+F 0 "C6" H 6542 1246 50  0000 L CNN
+F 1 "100n" H 6542 1155 50  0000 L CNN
+F 2 "Capacitor_SMD:C_0805_2012Metric" H 6450 1200 50  0001 C CNN
+F 3 "~" H 6450 1200 50  0001 C CNN
+	1    6450 1200
+	1    0    0    -1
+$EndComp
+Wire Wire Line
+	6450 1100 6100 1100
+Connection ~ 6100 1100
+Wire Wire Line
+	6450 1300 6100 1300
+Connection ~ 6100 1300
+Text Notes 5250 850  0    50   ~ 0
 RAM decoupling
-Text Notes 4800 850  0    50   ~ 0
+Text Notes 6050 850  0    50   ~ 0
 CPLD decoupling
 $Comp
@@
 L Device:C_Small C7
 U 1 1 5E9C1307
-P 5600 1200
-F 0 "C7" H 5692 1246 50  0000 L CNN
-F 1 "100n" H 5692 1155 50  0000 L CNN
-F 2 "Capacitor_SMD:C_0805_2012Metric" H 5600 1200 50  0001 C CNN
-F 3 "~" H 5600 1200 50  0001 C CNN
-	1    5600 1200
-	1    0    0    -1
-$EndComp
-Wire Wire Line
-	5200 1100 5600 1100
-Connection ~ 5200 1100
-Wire Wire Line
-	5600 1300 5200 1300
-Connection ~ 5200 1300
+P 6850 1200
+F 0 "C7" H 6942 1246 50  0000 L CNN
+F 1 "100n" H 6942 1155 50  0000 L CNN
+F 2 "Capacitor_SMD:C_0805_2012Metric" H 6850 1200 50  0001 C CNN
+F 3 "~" H 6850 1200 50  0001 C CNN
+	1    6850 1200
+	1    0    0    -1
+$EndComp
+Wire Wire Line
+	6450 1100 6850 1100
+Connection ~ 6450 1100
+Wire Wire Line
+	6850 1300 6450 1300
+Connection ~ 6450 1300
 Text Label 5150 4500 0    50   ~ 0
 TDI
@@
 F 0 "FID1" H 10885 6446 50  0000 L CNN
 F 1 "License" H 10885 6355 50  0000 L CNN
-F 2 "Sassa:CC_BY_SA_long_silkscreen_14x5.5mm" H 10800 6400 50  0001 C CNN
+F 2 "Sassa:CC_BY_NC_SA_square_silkscreen" H 10800 6400 50  0001 C CNN
 F 3 "~" H 10800 6400 50  0001 C CNN
 	1    10800 6400
@@
 	0    1    1    0
 $EndComp
+$Comp
+L Regulator_Linear:XC6206PxxxMR U11
+U 1 1 5FB507A7
+P 4450 1100
+F 0 "U11" H 4450 1342 50  0000 C CNN
+F 1 "XC6206PxxxMR" H 4450 1251 50  0000 C CNN
+F 2 "Package_TO_SOT_SMD:SOT-23" H 4450 1325 50  0001 C CIN
+F 3 "https://www.torexsemi.com/file/xc6206/XC6206.pdf" H 4450 1100 50  0001 C CNN
+	1    4450 1100
+	1    0    0    -1
+$EndComp
+$Comp
+L power:GND #PWR0102
+U 1 1 5FB5411A
+P 4450 1400
+F 0 "#PWR0102" H 4450 1150 50  0001 C CNN
+F 1 "GND" H 4455 1227 50  0000 C CNN
+F 2 "" H 4450 1400 50  0001 C CNN
+F 3 "" H 4450 1400 50  0001 C CNN
+	1    4450 1400
+	1    0    0    -1
+$EndComp
+$Comp
+L power:+3.3V #PWR0103
+U 1 1 5FB54A58
+P 4850 1100
+F 0 "#PWR0103" H 4850 950 50  0001 C CNN
+F 1 "+3.3V" H 4865 1273 50  0000 C CNN
+F 2 "" H 4850 1100 50  0001 C CNN
+F 3 "" H 4850 1100 50  0001 C CNN
+	1    4850 1100
+	1    0    0    -1
+$EndComp
+$Comp
+L power:+5V #PWR0104
+U 1 1 5FB55425
+P 4050 1100
+F 0 "#PWR0104" H 4050 950 50  0001 C CNN
+F 1 "+5V" H 4065 1273 50  0000 C CNN
+F 2 "" H 4050 1100 50  0001 C CNN
+F 3 "" H 4050 1100 50  0001 C CNN
+	1    4050 1100
+	1    0    0    -1
+$EndComp
+Wire Wire Line
+	4750 1100 4850 1100
+Wire Wire Line
+	4050 1100 4150 1100
+Text Notes 4100 750  0    50   ~ 0
+alternative footprint
+$Comp
+L Mechanical:Fiducial FID2
+U 1 1 5FCA38BE
+P 10250 6400
+F 0 "FID2" H 10335 6446 50  0000 L CNN
+F 1 "Logo" H 10335 6355 50  0000 L CNN
+F 2 "Sassa:PIC_Cassepanards_GS" H 10250 6400 50  0001 C CNN
+F 3 "~" H 10250 6400 50  0001 C CNN
+	1    10250 6400
+	1    0    0    -1
+$EndComp
 $EndSCHEMATC
